File: Schematic/VoiceRecognition.brd (EAGLE design)
At the start: 106.7 x 63.5 mm, 28 parts, among them Q1 16MHz, X1 USB-A

Commit message: PCB Schematic completed
Parts:
- removed IC1: (no value), adafruit:TO92-INLINE
- added !HWB, D+, D-, FUNC_GRN, GND_BARREL, GND_ICSP, MIC_SIGNAL, MISO, MOSI, NOFUNC_RED, PWR_BLU, RESET, SCK, SERVO_SIGNAL, TP4, TP7, VCC, VCC_TO_MIC, V_BARREL, V_ICSP, WARN_YELL: TPTP15SQ, testpad:TP15SQ
- added C12, C8: 100nF, rcl:C1206
- added J1: 5.5x2.1mm Barrel, SparkFun-Connectors:POWER_JACK_SMD
- added R8: 10k, rcl:M1206
- C3: value 100nF -> 1uF
- C6: value 1uF -> 100nF
- C7: value 1uF -> 10uF
- R3: value 150\ -> 1k
- R5: value 150 -> 1k
- R6: value 90 -> 1k
- R7: value 100 -> 1k
- moved C7 228.7 mm to (1.27, -219.7)
- moved MIC_ON 196.8 mm to (2.54, -207.0)
- moved C6 114.3 mm to (1.27, -88.9)
Connections:
- removed net FUNC-GRN: LED2.A
- removed net N$10: C6.1, IC1.2, X1.1
- removed net N$11: MIC_ON.P$2
- removed net N$4: JP1.3, U$1.9
- removed net NOFUNC-RED: LED3.A
- removed net WARN: LED4.A
- new net FUNC_GRN: FUNC_GRN.TP, LED2.A, U$1.28
- new net MIC_SIGNAL: JP2.1, MIC_SIGNAL.TP, U$1.41
- new net N$14: C8.1, U$1.42
- new net N$20: D-.TP, R2.2, U$1.3
- new net NOFUNC_RED: LED3.A, NOFUNC_RED.TP, U$1.30
- new net SERVO_POS: J1.VIN0, JP3.1, V_BARREL.TP
- new net WARN_YELL: LED4.A, U$1.29, WARN_YELL.TP
- net GND: now also C12.2, C8.2, GND_BARREL.TP, GND_ICSP.TP, J1.GND, J1.P$4, TP7.TP; no longer IC1.1, MIC_ON.P$1
- net HWB: now also !HWB.TP
- net N$12: now also D+.TP
- net N$13: now also MOSI.TP
- net N$15: now also C7.1, JP2.2, MIC_ON.P$2, VCC_TO_MIC.TP; no longer JP2.1, U$1.41
- net N$17: now also MISO.TP
- net N$2: now also JP1.3, SCK.TP, U$1.9; no longer R2.2, U$1.3
- net RST: now also R8.1, RESET.TP, TP4.TP
- net SIGNAL: now also SERVO_SIGNAL.TP, U$1.8
- net VCC: now also C12.1, C6.1, MIC_ON.P$1, PWR_BLU.TP, R8.2, VCC.TP, V_ICSP.TP, X1.1; no longer C7.1, IC1.3, JP2.2, JP3.1
